Commit message: Modular xacro improvements

File: urdf/gazebo_tags/gazebo_plugins.xacro (robot description, xacro)
@@ -11,6 +11,6 @@
             <wheel_radius>0.068</wheel_radius>
             <!--Best to use prefixes for frame ID's ('robotname/odom' for example) and to set the prefix on the RVIZ config too-->
-            <frame_id>carpet_rover/odom</frame_id>
-            <child_frame_id>carpet_rover/base_footprint</child_frame_id>
+            <frame_id>${robot_name}/odom</frame_id>
+            <child_frame_id>${robot_name}/base_footprint</child_frame_id>
         </plugin>
     </gazebo>

File: urdf/modules/carpet_rover.xacro (robot description, xacro)
@@ -28,5 +28,5 @@
       <origin xyz="0 0 0" rpy="0 0 0"/>
       <geometry>
-        <mesh filename="package://carpet_rover_description/assets/chassis_collision.stl"/>
+        <mesh filename="package://${package_name}/assets/chassis_collision.stl"/>
       </geometry>
     </collision>
@@ -35,5 +35,5 @@
       <origin xyz="-0.0455 -2.77556e-17 0.058" rpy="0 -0 1.5708"/>
       <geometry>
-        <mesh filename="package://carpet_rover_description/assets/raspi5.stl"/>
+        <mesh filename="package://${package_name}/assets/raspi5.stl"/>
       </geometry>
       <material name="raspi5_material">
@@ -45,5 +45,5 @@
       <origin xyz="0 1.26293e-18 0" rpy="0 -0 3.14159"/>
       <geometry>
-        <mesh filename="package://carpet_rover_description/assets/robotchassis.stl"/>
+        <mesh filename="package://${package_name}/assets/robotchassis.stl"/>
       </geometry>
       <material name="robotchassis_material">
@@ -55,5 +55,5 @@
       <origin xyz="0.0296 0.0215 0.05125" rpy="1.5708 -5.77779e-34 3.14159"/>
       <geometry>
-        <mesh filename="package://carpet_rover_description/assets/l298n.stl"/>
+        <mesh filename="package://${package_name}/assets/l298n.stl"/>
       </geometry>
       <material name="l298n_material">
@@ -65,5 +65,5 @@
       <origin xyz="0.00712895 0.0243036 0.0183344" rpy="1.13798e-15 1.5708 0"/>
       <geometry>
-        <mesh filename="package://carpet_rover_description/assets/dcmotor_motor.stl"/>
+        <mesh filename="package://${package_name}/assets/dcmotor_motor.stl"/>
       </geometry>
       <material name="dcmotor_motor_material">
@@ -75,5 +75,5 @@
       <origin xyz="0.00843232 0.0243036 0.0183344" rpy="1.26648e-15 1.5708 0"/>
       <geometry>
-        <mesh filename="package://carpet_rover_description/assets/dcmotor_belt.stl"/>
+        <mesh filename="package://${package_name}/assets/dcmotor_belt.stl"/>
       </geometry>
       <material name="dcmotor_belt_material">
@@ -85,5 +85,5 @@
       <origin xyz="0.00828145 0.0243036 0.0180594" rpy="1.13798e-15 1.5708 0"/>
       <geometry>
-        <mesh filename="package://carpet_rover_description/assets/dcmotor_body.stl"/>
+        <mesh filename="package://${package_name}/assets/dcmotor_body.stl"/>
       </geometry>
       <material name="dcmotor_body_material">
@@ -95,5 +95,5 @@
       <origin xyz="0.00712895 -0.0243036 -0.00833437" rpy="3.14159 -1.5708 0"/>
       <geometry>
-        <mesh filename="package://carpet_rover_description/assets/dcmotor_motor.stl"/>
+        <mesh filename="package://${package_name}/assets/dcmotor_motor.stl"/>
       </geometry>
       <material name="dcmotor_motor_2_material">
@@ -105,5 +105,5 @@
       <origin xyz="0.00843232 -0.0243036 -0.00833437" rpy="3.14159 -1.5708 0"/>
       <geometry>
-        <mesh filename="package://carpet_rover_description/assets/dcmotor_belt.stl"/>
+        <mesh filename="package://${package_name}/assets/dcmotor_belt.stl"/>
       </geometry>
       <material name="dcmotor_belt_2_material">
@@ -115,5 +115,5 @@
       <origin xyz="0.00828145 -0.0243036 -0.00805937" rpy="3.14159 -1.5708 0"/>
       <geometry>
-        <mesh filename="package://carpet_rover_description/assets/dcmotor_body.stl"/>
+        <mesh filename="package://${package_name}/assets/dcmotor_body.stl"/>
       </geometry>
       <material name="dcmotor_body_2_material">
@@ -125,5 +125,5 @@
       <origin xyz="-0.00712895 0.0243036 -0.00833437" rpy="-0 -1.5708 0"/>
       <geometry>
-        <mesh filename="package://carpet_rover_description/assets/dcmotor_motor.stl"/>
+        <mesh filename="package://${package_name}/assets/dcmotor_motor.stl"/>
       </geometry>
       <material name="dcmotor_motor_3_material">
@@ -135,5 +135,5 @@
       <origin xyz="-0.00843232 0.0243036 -0.00833437" rpy="1.28498e-16 -1.5708 0"/>
       <geometry>
-        <mesh filename="package://carpet_rover_description/assets/dcmotor_belt.stl"/>
+        <mesh filename="package://${package_name}/assets/dcmotor_belt.stl"/>
       </geometry>
       <material name="dcmotor_belt_3_material">
@@ -145,5 +145,5 @@
       <origin xyz="-0.00828145 0.0243036 -0.00805937" rpy="-1.13798e-15 -1.5708 0"/>
       <geometry>
-        <mesh filename="package://carpet_rover_description/assets/dcmotor_body.stl"/>
+        <mesh filename="package://${package_name}/assets/dcmotor_body.stl"/>
       </geometry>
       <material name="dcmotor_body_3_material">
@@ -155,5 +155,5 @@
       <origin xyz="-0.00712895 -0.0243036 0.0183344" rpy="-3.14159 1.5708 0"/>
       <geometry>
-        <mesh filename="package://carpet_rover_description/assets/dcmotor_motor.stl"/>
+        <mesh filename="package://${package_name}/assets/dcmotor_motor.stl"/>
       </geometry>
       <material name="dcmotor_motor_4_material">
@@ -165,5 +165,5 @@
       <origin xyz="-0.00843232 -0.0243036 0.0183344" rpy="-3.14159 1.5708 0"/>
       <geometry>
-        <mesh filename="package://carpet_rover_description/assets/dcmotor_belt.stl"/>
+        <mesh filename="package://${package_name}/assets/dcmotor_belt.stl"/>
       </geometry>
       <material name="dcmotor_belt_4_material">
@@ -175,5 +175,5 @@
       <origin xyz="-0.00828145 -0.0243036 0.0180594" rpy="-3.14159 1.5708 0"/>
       <geometry>
-        <mesh filename="package://carpet_rover_description/assets/dcmotor_body.stl"/>
+        <mesh filename="package://${package_name}/assets/dcmotor_body.stl"/>
       </geometry>
       <material name="dcmotor_body_4_material">
@@ -192,5 +192,5 @@
       <origin xyz="0 0 0.039" rpy="0 0 0"/>
       <geometry>
-        <mesh filename="package://carpet_rover_description/assets/wheel_collision.stl"/>
+        <mesh filename="package://${package_name}/assets/wheel_collision.stl"/>
       </geometry>
     </collision>
@@ -199,5 +199,5 @@
       <origin xyz="-0.0130594 -0.0592186 0.0251264" rpy="-1.5708 -5.28658e-33 -1.28245e-17"/>
       <geometry>
-        <mesh filename="package://carpet_rover_description/assets/dcmotor_axle.stl"/>
+        <mesh filename="package://${package_name}/assets/dcmotor_axle.stl"/>
       </geometry>
       <material name="dcmotor_axle_material">
@@ -209,5 +209,5 @@
       <origin xyz="0.032165 0.0313583 0.0494434" rpy="-3.14159 1.5708 0"/>
       <geometry>
-        <mesh filename="package://carpet_rover_description/assets/tyre.stl"/>
+        <mesh filename="package://${package_name}/assets/tyre.stl"/>
       </geometry>
       <material name="tyre_material">
@@ -219,5 +219,5 @@
       <origin xyz="0.032165 0.0313583 0.0494334" rpy="-3.14159 1.5708 0"/>
       <geometry>
-        <mesh filename="package://carpet_rover_description/assets/wheel.stl"/>
+        <mesh filename="package://${package_name}/assets/wheel.stl"/>
       </geometry>
       <material name="wheel_material">
@@ -244,5 +244,5 @@
       <origin xyz="0 0 0.039" rpy="0 0 0"/>
       <geometry>
-        <mesh filename="package://carpet_rover_description/assets/wheel_collision.stl"/>
+        <mesh filename="package://${package_name}/assets/wheel_collision.stl"/>
       </geometry>
     </collision>
@@ -251,5 +251,5 @@
       <origin xyz="-0.0130594 -0.0592186 0.0251264" rpy="-1.5708 6.48832e-32 -3.01686e-17"/>
       <geometry>
-        <mesh filename="package://carpet_rover_description/assets/dcmotor_axle.stl"/>
+        <mesh filename="package://${package_name}/assets/dcmotor_axle.stl"/>
       </geometry>
       <material name="dcmotor_axle_2_material">
@@ -261,5 +261,5 @@
       <origin xyz="0.032165 0.0313583 0.0494434" rpy="-3.14159 1.5708 0"/>
       <geometry>
-        <mesh filename="package://carpet_rover_description/assets/tyre.stl"/>
+        <mesh filename="package://${package_name}/assets/tyre.stl"/>
       </geometry>
       <material name="tyre_2_material">
@@ -271,5 +271,5 @@
       <origin xyz="0.032165 0.0313583 0.0494334" rpy="-3.14159 1.5708 0"/>
       <geometry>
-        <mesh filename="package://carpet_rover_description/assets/wheel.stl"/>
+        <mesh filename="package://${package_name}/assets/wheel.stl"/>
       </geometry>
       <material name="wheel_2_material">
@@ -296,5 +296,5 @@
       <origin xyz="0 0 0.039" rpy="0 0 0"/>
       <geometry>
-        <mesh filename="package://carpet_rover_description/assets/wheel_collision.stl"/>
+        <mesh filename="package://${package_name}/assets/wheel_collision.stl"/>
       </geometry>
     </collision>
@@ -303,5 +303,5 @@
       <origin xyz="-0.0130594 -0.0592186 0.0251264" rpy="-1.5708 8.78702e-32 -2.07236e-17"/>
       <geometry>
-        <mesh filename="package://carpet_rover_description/assets/dcmotor_axle.stl"/>
+        <mesh filename="package://${package_name}/assets/dcmotor_axle.stl"/>
       </geometry>
       <material name="dcmotor_axle_3_material">
@@ -313,5 +313,5 @@
       <origin xyz="0.032165 0.0313583 0.0494434" rpy="-3.14159 1.5708 0"/>
       <geometry>
-        <mesh filename="package://carpet_rover_description/assets/tyre.stl"/>
+        <mesh filename="package://${package_name}/assets/tyre.stl"/>
       </geometry>
       <material name="tyre_3_material">
@@ -323,5 +323,5 @@
       <origin xyz="0.032165 0.0313583 0.0494334" rpy="-3.14159 1.5708 0"/>
       <geometry>
-        <mesh filename="package://carpet_rover_description/assets/wheel.stl"/>
+        <mesh filename="package://${package_name}/assets/wheel.stl"/>
       </geometry>
       <material name="wheel_3_material">
@@ -348,5 +348,5 @@
       <origin xyz="0 0 0.039" rpy="0 0 0"/>
       <geometry>
-        <mesh filename="package://carpet_rover_description/assets/wheel_collision.stl"/>
+        <mesh filename="package://${package_name}/assets/wheel_collision.stl"/>
       </geometry>
     </collision>
@@ -355,5 +355,5 @@
       <origin xyz="-0.0130594 -0.0592186 0.0251264" rpy="-1.5708 -1.43421e-33 2.55822e-17"/>
       <geometry>
-        <mesh filename="package://carpet_rover_description/assets/dcmotor_axle.stl"/>
+        <mesh filename="package://${package_name}/assets/dcmotor_axle.stl"/>
       </geometry>
       <material name="dcmotor_axle_4_material">
@@ -365,5 +365,5 @@
       <origin xyz="0.032165 0.0313583 0.0494434" rpy="-3.14159 1.5708 0"/>
       <geometry>
-        <mesh filename="package://carpet_rover_description/assets/tyre.stl"/>
+        <mesh filename="package://${package_name}/assets/tyre.stl"/>
       </geometry>
       <material name="tyre_4_material">
@@ -375,5 +375,5 @@
       <origin xyz="0.032165 0.0313583 0.0494334" rpy="-3.14159 1.5708 0"/>
       <geometry>
-        <mesh filename="package://carpet_rover_description/assets/wheel.stl"/>
+        <mesh filename="package://${package_name}/assets/wheel.stl"/>
       </geometry>
       <material name="wheel_4_material">

File: urdf/robot.urdf.xacro (robot description, xacro)
@@ -1,4 +1,5 @@
 <?xml version="1.0" ?>
 <robot name="carpet_rover" xmlns:xacro="http://www.ros.org/wiki/xacro">
+    <xacro:include filename="xacro_properties/xacro_properties.xacro" />
     <xacro:include filename="modules/carpet_rover.xacro" />
     <xacro:include filename="gazebo_tags/gazebo_plugins.xacro" />
